File: Hello_World/Hello_World.kicad_pcb (KiCad board)
At the start: 8 copper layers, 179 x 47 mm, 10 parts, among them P1 Nokia 5110/3310 Monochrome LCD, P2 CONN_1, P3 CONN_1, T1 Touch Sensor, U1 FEATHER_M0_EXPRESS, U2 MPR121_BREAKOUT

Commit message: Final tweaks to the Hello World circuit.
Parts:
- T1: value Touch Sensor -> us mx br it de ru na ir cn fr jp in
Routing:
- net GND: track 482.8 -> 481.9 mm
