File: Hello_World/Hello_World.sch (KiCad schematic (older format))
At the start: 0 parts

Commit message: (Re-)Initialize project
Parts:
- added P1: Nokia 5110/3310 Monochrome LCD, ~, symbol CONN_8
- added P2, P3: CONN_1, ~, symbol CONN_1
- added T1: Touch Sensor, ~, symbol CONN_12
- added U1: FEATHER_M0_EXPRESS, ~, symbol FEATHER_M0_EXPRESS
- added U2: MPR121_BREAKOUT, ~, symbol MPR121_BREAKOUT
Connections:
- new net: U1.17 (SDA), U2.18 (SDA)
- new net: U1.18 (SCL), U2.19 (SCL)
- new net: T1.12 (P12), U2.1 (#11)
- new net: T1.3 (P3), U2.10 (#2)
- new net: T1.2 (P2), U2.11 (#1)
- new net: T1.1 (P1), U2.12 (#0)
- new net: T1.11 (P11), U2.2 (#10)
- new net: T1.10 (P10), U2.3 (#9)
- new net: T1.9 (P9), U2.4 (#8)
- new net: T1.8 (P8), U2.5 (#7)
- new net: T1.7 (P7), U2.6 (#6)
- new net: T1.6 (P6), U2.7 (#5)
- new net: T1.5 (P5), U2.8 (#4)
- new net: T1.4 (P4), U2.9 (#3)
- new net +3.3V: P1.2 (P2), P3.1, U1.2 (3V), U2.14 (Vin)
- new net CLK: P1.3 (P3), U1.11 (SCK)
- new net CS: P1.6 (P6), U1.22 (10~)
- new net DIN: P1.4 (P4), U1.12 (MOSI)
- new net D_C: P1.5 (P5), U1.23 (11~)
- new net GND: P1.1 (P1), P2.1, U1.16 (GND), U1.4 (GND), U2.13 (GND), U2.16 (GND), U2.17 (Addr)
- new net LED: P1.8 (P8), U1.19 (~5)
- new net RST: P1.7 (P7), U1.20 (6)

Commit message: Final tweaks to the Hello World circuit.
Parts:
- T1: value Touch Sensor -> us mx br it de ru na ir cn fr jp in
Changed lines of the file:
@@
 LIBS:feather_m0_express
 LIBS:metromini
+LIBS:Hello_World-cache
 EELAYER 27 0
 EELAYER END
@@
 Sheet 1 1
 Title ""
-Date "22 oct 2018"
+Date "24 oct 2018"
 Rev ""
 Comp ""
@@
 P 7450 2650
 F 0 "T1" V 7400 2650 60  0000 C CNN
-F 1 "Touch Sensor" V 7500 2650 60  0000 C CNN
+F 1 "us mx br it de ru na ir cn fr jp in" V 7500 2650 60  0000 C CNN
 F 2 "~" H 7450 2650 60  0000 C CNN
 F 3 "~" H 7450 2650 60  0000 C CNN
