File: WhyDidTheChicken/WhyDidTheChicken.kicad_pcb (KiCad board)
At the start: 8 copper layers, 179 x 47 mm, 4 parts

Commit message: Complete two more: WelcomeToGothemCity and WhyDidTheChicken
Parts:
- added P1: PedSignal, PIN_ARRAY_4x1, F.Cu at (118.1, 86.4)
- added P2: LEDS+Button, pin_array_6x1, F.Cu at (102.9, 86.4)
- added P3: CONN_1, PIN_ARRAY_1, F.Cu at (185.4, 55.9)
- added P4: CONN_1, PIN_ARRAY_1, F.Cu at (195.6, 94.0)
- added P5: CONN_1, PIN_ARRAY_1, F.Cu at (195.6, 96.5)
- added R1: 150 Ohms, R4, F.Cu at (99.1, 76.2)
- added R2: 150 Ohms, R4, F.Cu at (104.1, 76.2)
- added R3: 150 Ohms, R4, F.Cu at (101.6, 76.2)
- added U1: ADAFRUIT_POWERBOOST_500, PBost500Breakout, F.Cu at (142.2, 78.1)
- added U2: METROMINI, MetroMini, F.Cu at (184.2, 78.7)
Routing:
- net (no net): track 2486.7 -> 1427.5 mm, vias 1236 -> 785
- net GND: track 0.00 -> 455.1 mm, vias 0 -> 160
- net +5V: track 0.00 -> 428.4 mm, vias 0 -> 140
- net /Vin: track 0.00 -> 197.7 mm, vias 0 -> 74
- net N-0000010: track 0.00 -> 156.1 mm, vias 0 -> 12
- net N-000009: track 0.00 -> 139.2 mm, vias 0 -> 10
- net N-000008: track 0.00 -> 133.1 mm, vias 0 -> 10
- net /Walk: track 0.00 -> 105.1 mm, vias 0 -> 10
- net /SCL: track 0.00 -> 92.5 mm, vias 0 -> 10
- net /SDA: track 0.00 -> 92.4 mm, vias 0 -> 10
- net /Yellow: track 0.00 -> 10.2 mm, vias 0 -> 5
- net /Red: track 0.00 -> 10.2 mm, vias 0 -> 5
- net /Green: track 0.00 -> 10.2 mm, vias 0 -> 5
