File: SprocketFactory/SprocketFactory.kicad_pcb (KiCad board)
At the start: 8 copper layers, 179 x 47 mm, 4 parts

Commit message: Completed SprocketFactory
Parts:
- removed ? (x4): , MH
- added SW1: Start, SW_PUSH-12mm, F.Cu at (241.9, 139.1)
- added SW2: Stop, SW_PUSH-12mm, F.Cu at (241.9, 160.0)
- added U1: FEATHER_M0_EXPRESS, AdafruitFeather, F.Cu at (201.9, 133.3)
- added U2: 8-CHANNELSERVO​FEATHERWING, 8ChanPWMWing, F.Cu at (201.9, 133.3)
- added U3: ADAFRUIT_POWERBOOST_500, PBost500Breakout, F.Cu at (236.2, 95.2)
Routing:
- net (no net): track 2486.7 -> 0.00 mm, vias 1236 -> 0
- net /GND: track 0.00 -> 224.4 mm
- net /5: track 0.00 -> 42.6 mm
- net /6: track 0.00 -> 40.3 mm
- net /BAT: track 0.00 -> 36.1 mm
- net N-000003: track 0.00 -> 21.2 mm
Other:
- board outline removed
- copper layers 8 -> 2
- rule pad_to_mask_clearance: 0 -> 0.2
