File: SprocketFactory/SprocketFactory.sch (KiCad schematic (older format))
At the start: 5 parts, among them SW1 Start, SW2 Stop, U1 FEATHER_M0_EXPRESS, U2 8-CHANNELSERVO​FEATHERWING, U3 ADAFRUIT_POWERBOOST_500

Commit message: Add detailed comments to both the code and the schematics
Other:
- note added: "U1 (Feather M0 Express) and U2 (8-channel PWM/Servo FeatherWing)\nare stacked. The 8 servos are not shown, but are connected to the \nservo headers on the 8-channel PWM/Servo FeatherWing. U2 has \nconnect points for all I/O and power pins and these holes are used to \nconnect the Power Boost 1000c and the Start and Stop switches. The\nbattery is plugged into the Power Boost and not the Feather, s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"
Changed lines of the file:
@@
 Sheet 1 1
 Title ""
-Date "29 oct 2018"
+Date "11 nov 2018"
 Rev ""
 Comp ""
@@
 Connection ~ 7350 2550
 Connection ~ 7500 750
+Text Notes 2550 3500 0    60   ~ 0
+U1 (Feather M0 Express) and U2 (8-channel PWM/Servo FeatherWing)\nare stacked.  The 8 servos are not shown, but are connected to the \nservo headers on the 8-channel PWM/Servo FeatherWing.  U2 has \nconnect points for all I/O and power pins and these holes are used to \nconnect the Power Boost 1000c and the Start and Stop switches.  The\nbattery is plugged into the Power Boost and not the Feather, since the\nServos can be power hungry and want all of 5V to work well.
 $EndSCHEMATC
