File: WelcomeToGothemCity/WelcomeToGothemCity.sch (KiCad schematic (older format))
At the start: 0 parts

Commit message: Complete Welcome To Gothem City
Parts:
- added P1: HC-SR04, ~, symbol CONN_4
- added P2: LEDS, ~, symbol CONN_2
- added P3, P4, P5: CONN_1, ~, symbol CONN_1
- added Q1: TIP120, TO220, symbol TIP120
- added R1: 1K Ohms, ~, symbol R
- added R2: R, ~, symbol R
- added U1: ADAFRUIT_POWERBOOST_500, ~, symbol ADAFRUIT_POWERBOOST_500
- added U2: METROMINI, ~, symbol METROMINI
Connections:
- new net: U1.8 (5V), U2.22 (Vin)
- new net: R1.1, U2.9 (#5)
- new net: Q1.1 (B), R1.2
- new net: Q1.2 (C), R2.2
- new net: P2.2 (PM), R2.1
- new net +5V: P1.1 (P1), P4.1, U2.25 (5V)
- new net +BATT: P2.1 (P1), P3.1, U1.3 (BATT)
- new net Echo: P1.3 (P3), U2.7 (#7)
- new net GND: P1.4 (P4), P5.1, Q1.3 (E), U1.2 (GND), U1.5 (GND), U1.7 (GND), U2.23 (GND), U2.24 (GND)
- new net Trig: P1.2 (P2), U2.6 (#8)

Commit message: Update WelcomeToGothemCity: actual value for R2
Parts:
- R2: value R -> 2.7 Ohms, 3 Watt; Mouser Part Number (none) -> 594-5093NW2R700J
Changed lines of the file:
@@
 Sheet 1 1
 Title ""
-Date "25 oct 2018"
+Date "1 nov 2018"
 Rev ""
 Comp ""
@@
 P 4900 2400
 F 0 "R2" V 4980 2400 40  0000 C CNN
-F 1 "R" V 4907 2401 40  0000 C CNN
+F 1 "2.7 Ohms, 3 Watt" V 4907 2401 40  0000 C CNN
 F 2 "~" V 4830 2400 30  0000 C CNN
 F 3 "~" H 4900 2400 30  0000 C CNN
+F 4 "594-5093NW2R700J" H 4900 2400 60  0001 C CNN "Mouser Part Number"
 	1    4900 2400
 	1    0    0    -1
