File: OnlyHerHairdresser/OnlyHerHairdresser.sch (KiCad schematic (older format))
At the start: 0 parts

Commit message: OnlyHerHairdresser: circuit designed and board laid out
Parts:
- added P1: TCS34725 Breakout, ~, symbol CONN_7
- added P2: RGB LEDS, ~, symbol CONN_4
- added P3, P4, P5: CONN_1, ~, symbol CONN_1
- added Q1: MPQ3904, ~, symbol MPQ3904
- added R1, R3, R5: 1K Ohms, ~, symbol R
- added R2, R4, R6: 45 Ohms, ~, symbol R
- added SW1: SW_PUSH, ~, symbol SW_PUSH
- added U1: FEATHER_M0_EXPRESS, ~, symbol FEATHER_M0_EXPRESS
Connections:
- new net: R5.1, U1.19 (~5)
- new net: R3.1, U1.20 (6)
- new net: R1.1, U1.22 (10~)
- new net: SW1.1, U1.23 (11~)
- new net: Q1.1 (C), R2.2
- new net: Q1.2 (B), R1.2
- new net: Q1.6 (B), R3.2
- new net: Q1.7 (C), R4.2
- new net: Q1.8 (C), R6.2
- new net: Q1.9 (B), R5.2
- new net 3V3: P1.5 (P5)
- new net B: P2.3 (P3), R6.1
- new net Comm: P2.4 (P4), P5.1, U1.28 (BAT)
- new net G: P2.2 (P2), R4.1
- new net GND: P1.6 (P6), P3.1, Q1.10 (E), Q1.3 (E), Q1.5 (E), SW1.2, U1.16 (GND), U1.4 (GND)
- new net INT: P1.1 (P1), P1.2 (P2)
- new net R: P2.1 (P1), R2.1
- new net SCL: P1.4 (P4), U1.18 (SCL)
- new net SDA: P1.3 (P3), U1.17 (SDA)
- new net VIN: P1.7 (P7), P4.1, U1.2 (3V)
