File: SteelWheels/SteelWheels.kicad_pcb (KiCad board)
At the start: 8 copper layers, 179 x 47 mm, 4 parts

Commit message: Completed SteelWheels
Parts:
- added T1: Throttle, PIN_ARRAY_3X1, F.Cu at (111.8, 66.0)
- added T2: Neopixels, PIN_ARRAY_3X1, F.Cu at (111.8, 88.9)
- added U1: ADAFRUIT_POWERBOOST_1000, PBost500Breakout, F.Cu at (139.7, 78.2)
- added U2: METROMINI, MetroMini, F.Cu at (184.2, 78.7)
Routing:
- net (no net): track 2486.7 -> 1722.1 mm, vias 1236 -> 914
- net GND: track 0.00 -> 387.4 mm, vias 0 -> 152
- net +5V: track 0.00 -> 234.3 mm, vias 0 -> 75
- net +3.3V: track 0.00 -> 198.7 mm, vias 0 -> 75
- net N-000002: track 0.00 -> 92.5 mm, vias 0 -> 10
- net /ThrottleIn: track 0.00 -> 90.0 mm, vias 0 -> 10
